File: mPCIe-GNSS/mPCIe-GNSS.sch (KiCad schematic (older format))
At the start: 23 parts, among them J1 ANT, J2 IO, Q1 DTC143ZEBTL, Q2 DTC143ZEBTL, U1 LEA-M8T

Commit message: updoots
Parts:
- BAT1: footprint 1 My Footprints:CAP_DSK-3R3H224U-HL -> mPCIe-GNSS:CAP_DSK-3R3H224U-HL
- J1: footprint 1 My Footprints:U.FL_Hirose_U.FL-R-SMT-1_Vertical_Tweaked -> mPCIe-GNSS:U.FL_Hirose_U.FL-R-SMT-1_Vertical_Tweaked
- J2: footprint 1 My Footprints:JST_SH_SM06B-SRSS-TB_1x06-1MP_P1.00mm_Horizontal_3D -> mPCIe-GNSS:JST_SH_SM06B-SRSS-TB_1x06-1MP_P1.00mm_Horizontal_3D
- LED1, LED2, LED3: footprint 1 My Footprints:LED_0603_1608Metric_SnapModel -> mPCIe-GNSS:LED_0603_1608Metric_SnapModel
- Q1, Q2: footprint 1 My Footprints:Q_EMT3F -> mPCIe-GNSS:Q_EMT3F
- U1: footprint 1 My Footprints:ublox_LEA -> mPCIe-GNSS:ublox_LEA
Other:
- moved on the sheet: J2
Changed lines of the file:
@@
 F 0 "LED2" H 8843 5067 50  0000 C CNN
 F 1 "TP1" H 8843 4976 50  0000 C CNN
-F 2 "1 My Footprints:LED_0603_1608Metric_SnapModel" H 8850 4850 50  0001 C CNN
+F 2 "mPCIe-GNSS:LED_0603_1608Metric_SnapModel" H 8850 4850 50  0001 C CNN
 F 3 "~" H 8850 4850 50  0001 C CNN
 F 4 "C72038" H 8850 4850 50  0001 C CNN "LCSC"
@@
 F 0 "LED1" H 8043 5067 50  0000 C CNN
 F 1 "PWR" H 8043 4976 50  0000 C CNN
-F 2 "1 My Footprints:LED_0603_1608Metric_SnapModel" H 8050 4850 50  0001 C CNN
+F 2 "mPCIe-GNSS:LED_0603_1608Metric_SnapModel" H 8050 4850 50  0001 C CNN
 F 3 "~" H 8050 4850 50  0001 C CNN
 F 4 "C72041" H 8050 4850 50  0001 C CNN "LCSC"
@@
 F 0 "Q1" V 8600 5800 50  0000 L CNN
 F 1 "DTC143ZEBTL" V 8700 5800 50  0000 L CNN
-F 2 "1 My Footprints:Q_EMT3F" H 8800 5700 50  0001 C CNN
+F 2 "mPCIe-GNSS:Q_EMT3F" H 8800 5700 50  0001 C CNN
 F 3 "~" H 8800 5700 50  0001 C CNN
 F 4 "C172398" H 8800 5700 50  0001 C CNN "LCSC"
@@
 F 0 "J1" H 7200 2425 50  0000 L CNN
 F 1 "ANT" H 7200 2334 50  0000 L CNN
-F 2 "1 My Footprints:U.FL_Hirose_U.FL-R-SMT-1_Vertical_Tweaked" H 7100 2450 50  0001 C CNN
+F 2 "mPCIe-GNSS:U.FL_Hirose_U.FL-R-SMT-1_Vertical_Tweaked" H 7100 2450 50  0001 C CNN
 F 3 " ~" H 7100 2450 50  0001 C CNN
 F 4 "" H 7100 2450 50  0001 C CNN "LCSC"
@@
 Text Label 3150 2250 0    50   ~ 0
 ~RESET
-Text Label 5550 4800 2    50   ~ 0
+Text Label 5550 4850 2    50   ~ 0
 TXD
 NoConn ~ 2750 1350
@@
 F 0 "LED3" H 9643 5067 50  0000 C CNN
 F 1 "TP2" H 9643 4976 50  0000 C CNN
-F 2 "1 My Footprints:LED_0603_1608Metric_SnapModel" H 9650 4850 50  0001 C CNN
+F 2 "mPCIe-GNSS:LED_0603_1608Metric_SnapModel" H 9650 4850 50  0001 C CNN
 F 3 "~" H 9650 4850 50  0001 C CNN
 F 4 "C2286" H 9650 4850 50  0001 C CNN "LCSC"
@@
 F 0 "Q2" V 9400 5800 50  0000 L CNN
 F 1 "DTC143ZEBTL" V 9500 5800 50  0000 L CNN
-F 2 "1 My Footprints:Q_EMT3F" H 9600 5700 50  0001 C CNN
+F 2 "mPCIe-GNSS:Q_EMT3F" H 9600 5700 50  0001 C CNN
 F 3 "~" H 9600 5700 50  0001 C CNN
 F 4 "C172398" H 9600 5700 50  0001 C CNN "LCSC"
@@
 L Connector:Conn_01x06_Female J2
 U 1 1 60033A72
-P 5950 4800
-F 0 "J2" H 5978 4776 50  0000 L CNN
-F 1 "IO" H 5978 4685 50  0000 L CNN
-F 2 "1 My Footprints:JST_SH_SM06B-SRSS-TB_1x06-1MP_P1.00mm_Horizontal_3D" H 5950 4800 50  0001 C CNN
-F 3 "~" H 5950 4800 50  0001 C CNN
-	1    5950 4800
-	1    0    0    -1
-$EndComp
-Text Label 5550 4700 2    50   ~ 0
+P 5950 4850
+F 0 "J2" H 5978 4826 50  0000 L CNN
+F 1 "IO" H 5978 4735 50  0000 L CNN
+F 2 "mPCIe-GNSS:JST_SH_SM06B-SRSS-TB_1x06-1MP_P1.00mm_Horizontal_3D" H 5950 4850 50  0001 C CNN
+F 3 "~" H 5950 4850 50  0001 C CNN
+	1    5950 4850
+	1    0    0    -1
+$EndComp
+Text Label 5550 4750 2    50   ~ 0
 TP1
-Text Label 5550 4900 2    50   ~ 0
+Text Label 5550 4950 2    50   ~ 0
 RXD
 Wire Wire Line
-	5550 4800 5750 4800
-Wire Wire Line
-	5750 5000 5550 5000
-Wire Wire Line
-	5750 4700 5550 4700
+	5550 4850 5750 4850
+Wire Wire Line
+	5750 5050 5550 5050
+Wire Wire Line
+	5750 4750 5550 4750
 Text Label 4800 2150 2    50   ~ 0
 TXD
@@
 Wire Wire Line
 	5000 2250 4800 2250
-Text Label 5550 5000 2    50   ~ 0
+Text Label 5550 5050 2    50   ~ 0
 TP2
 Wire Wire Line
-	5750 4600 5550 4600
-Wire Wire Line
-	5750 4900 5550 4900
-Text Label 5550 5100 2    50   ~ 0
-+3.3V
-Text Label 5550 4600 2    50   ~ 0
-GND
-Wire Wire Line
-	5750 5100 5550 5100
+	5750 4650 5550 4650
+Wire Wire Line
+	5750 4950 5550 4950
+Text Label 5550 5150 2    50   ~ 0
++3.3V
+Text Label 5550 4650 2    50   ~ 0
+GND
+Wire Wire Line
+	5750 5150 5550 5150
 $Comp
 L Device:C C1
@@
 F 0 "BAT1" H 8750 2500 50  0000 R CNN
 F 1 "DSK-3R3H224U" H 8750 2400 50  0000 R CNN
-F 2 "1 My Footprints:CAP_DSK-3R3H224U-HL" H 8888 2300 50  0001 C CNN
+F 2 "mPCIe-GNSS:CAP_DSK-3R3H224U-HL" H 8888 2300 50  0001 C CNN
 F 3 "~" H 8850 2450 50  0001 C CNN
 	1    8850 2450
@@
 F 0 "U1" H 5150 3550 50  0000 C CNN
 F 1 "LEA-M8T" H 5150 3450 50  0000 C CNN
-F 2 "1 My Footprints:ublox_LEA" H 5700 2450 50  0001 L BNN
+F 2 "mPCIe-GNSS:ublox_LEA" H 5700 2450 50  0001 L BNN
 F 3 "" H 5700 2450 50  0001 L BNN
 F 4 "2.7 mm" H 5700 2450 50  0001 L BNN "MAXIMUM_PACKAGE_HEIGHT"
